Commit message: feat: add a 2D lidar and a guard that stops the robot before obstacles

File: aruco_world/urdf/camera_bot.urdf.xacro (robot description, xacro)
@@ -1,9 +1,10 @@
 <?xml version="1.0"?>
 <!--
-  Generic differential drive robot with a forward-facing camera. Gazebo spawns the robot from this
-  description and robot_state_publisher turns it into TF.
+  Generic differential drive robot with a forward-facing camera and a 360-degree 2D lidar on a mast.
+  Gazebo spawns the robot from this description and robot_state_publisher turns it into TF.
   Frames follow REP 105 and REP 103: base_footprint on the floor under the wheel axle, base_link at
   the centre of the body, both with x forward, y left, z up. camera_link_optical is the camera's
-  optical frame (z forward, x right, y down): images and detections are stamped in it.
+  optical frame (z forward, x right, y down): images and detections are stamped in it. lidar_link
+  is the centre of the scan plane, and scans are stamped in it.
 -->
 <robot name="camera_bot" xmlns:xacro="http://www.ros.org/wiki/xacro">
@@ -23,4 +24,20 @@
   <xacro:property name="camera_z" value="0.25"/>  <!-- lens above the floor -->
   <xacro:property name="camera_mass" value="0.05"/>
+  <!-- The scan plane sits above the camera, so nothing on the robot blocks any direction. -->
+  <xacro:property name="lidar_z" value="0.30"/>
+  <xacro:property name="lidar_radius" value="0.025"/>
+  <xacro:property name="lidar_height" value="0.035"/>
+  <xacro:property name="lidar_mass" value="0.1"/>
+  <xacro:property name="mast_radius" value="0.01"/>
+  <!-- A low-cost 360-degree time-of-flight lidar, from the datasheets of two common ones: 5,000
+       samples per second at 10 turns per second, so 500 rays 0.72 degrees apart. Where they
+       differ, the less favourable value is used, so what works here should work with either. -->
+  <xacro:property name="lidar_rate" value="10"/>
+  <xacro:property name="lidar_samples" value="500"/>
+  <xacro:property name="lidar_range_min" value="0.05"/>
+  <xacro:property name="lidar_range_max" value="12.0"/>
+  <!-- The datasheets give +-3 cm without saying what it bounds; read here as three standard
+       deviations. -->
+  <xacro:property name="lidar_noise_stddev" value="0.01"/>
   <material name="body"><color rgba="0.15 0.35 0.6 1"/></material>
   <material name="dark"><color rgba="0.1 0.1 0.1 1"/></material>
@@ -69,4 +86,13 @@
       <origin xyz="0.15 0 0.09" rpy="0 0 0"/>
       <geometry><box size="0.03 0.03 0.10"/></geometry>
+      <material name="grey"/>
+    </visual>
+    <!-- Lidar mast, from the top of the body to the bottom of the lidar -->
+    <visual>
+      <origin xyz="0 0 ${(body_height / 2 + lidar_z - body_z - lidar_height / 2) / 2}" rpy="0 0 0"/>
+      <geometry>
+        <cylinder radius="${mast_radius}"
+                  length="${lidar_z - body_z - lidar_height / 2 - body_height / 2}"/>
+      </geometry>
       <material name="grey"/>
     </visual>
@@ -148,4 +174,56 @@
     </sensor>
   </gazebo>
+  <!-- ===================== Lidar ===================== -->
+  <joint name="lidar_joint" type="fixed">
+    <parent link="base_link"/>
+    <child link="lidar_link"/>
+    <origin xyz="0 0 ${lidar_z - body_z}" rpy="0 0 0"/>
+  </joint>
+  <!-- The housing is narrower than the minimum range, so the lidar never sees itself. -->
+  <link name="lidar_link">
+    <xacro:box_inertia mass="${lidar_mass}" x="${2 * lidar_radius}" y="${2 * lidar_radius}"
+                       z="${lidar_height}"/>
+    <visual>
+      <geometry><cylinder radius="${lidar_radius}" length="${lidar_height}"/></geometry>
+      <material name="dark"/>
+    </visual>
+  </link>
+  <gazebo reference="lidar_link">
+    <sensor name="lidar" type="gpu_lidar">
+      <always_on>true</always_on>
+      <update_rate>${lidar_rate}</update_rate>
+      <visualize>true</visualize>
+      <topic>/scan</topic>
+      <gz_frame_id>lidar_link</gz_frame_id>
+      <lidar>
+        <scan>
+          <horizontal>
+            <samples>${lidar_samples}</samples>
+            <resolution>1</resolution>
+            <!-- A full turn that does not measure the same direction twice: the last ray stops
+                 one step short of the first. -->
+            <min_angle>${-pi}</min_angle>
+            <max_angle>${pi - 2 * pi / lidar_samples}</max_angle>
+          </horizontal>
+          <vertical>
+            <samples>1</samples>
+            <resolution>1</resolution>
+            <min_angle>0</min_angle>
+            <max_angle>0</max_angle>
+          </vertical>
+        </scan>
+        <range>
+          <min>${lidar_range_min}</min>
+          <max>${lidar_range_max}</max>
+          <resolution>0.01</resolution>
+        </range>
+        <noise>
+          <type>gaussian</type>
+          <mean>0</mean>
+          <stddev>${lidar_noise_stddev}</stddev>
+        </noise>
+      </lidar>
+    </sensor>
+  </gazebo>
   <!-- ===================== Gazebo systems ===================== -->
   <gazebo>

Commit message: feat: place the robot in the map from the markers it sees
Wheels now collide as spheres: the cylinders touched the floor on their inner edges, so the odometry under-counted turns.

File: aruco_world/urdf/camera_bot.urdf.xacro (robot description, xacro)
@@ -118,6 +118,9 @@
         <material name="dark"/>
       </visual>
+      <!-- A sphere, not the cylinder: a cylinder touches the floor along its rim's edges, and
+           turning on the inner edges shrinks the wheel separation the odometry assumes. A sphere
+           touches at one point, right under the wheel's centre. -->
       <collision>
-        <geometry><cylinder radius="${wheel_radius}" length="${wheel_width}"/></geometry>
+        <geometry><sphere radius="${wheel_radius}"/></geometry>
       </collision>
     </link>
@@ -248,4 +251,15 @@
       <topic>/joint_states</topic>
     </plugin>
+    <!-- Ground truth, for checking estimates: the robot's true pose in the world, which is the map
+         frame. It goes to its own topics and never to /tf, so no node mistakes it for a sensor. -->
+    <plugin filename="gz-sim-odometry-publisher-system"
+            name="gz::sim::systems::OdometryPublisher">
+      <odom_frame>map</odom_frame>
+      <robot_base_frame>base_footprint</robot_base_frame>
+      <odom_topic>/ground_truth</odom_topic>
+      <tf_topic>/ground_truth/tf</tf_topic>
+      <odom_publish_frequency>30</odom_publish_frequency>
+      <dimensions>2</dimensions>
+    </plugin>
   </gazebo>
 </robot>

Commit message: feat: fuse drifting odometry, a gyro and the marker fixes with two robot_localization filters

File: aruco_world/urdf/camera_bot.urdf.xacro (robot description, xacro)
@@ -1,10 +1,11 @@
 <?xml version="1.0"?>
 <!--
-  Generic differential drive robot with a forward-facing camera and a 360-degree 2D lidar on a mast.
-  Gazebo spawns the robot from this description and robot_state_publisher turns it into TF.
+  Generic differential drive robot with a forward-facing camera, a 360-degree 2D lidar on a mast and
+  an IMU. Gazebo spawns the robot from this description and robot_state_publisher turns it into TF.
   Frames follow REP 105 and REP 103: base_footprint on the floor under the wheel axle, base_link at
   the centre of the body, both with x forward, y left, z up. camera_link_optical is the camera's
   optical frame (z forward, x right, y down): images and detections are stamped in it. lidar_link
-  is the centre of the scan plane, and scans are stamped in it.
+  is the centre of the scan plane, and scans are stamped in it. imu_link sits at the centre of the
+  body, aligned with it.
 -->
 <robot name="camera_bot" xmlns:xacro="http://www.ros.org/wiki/xacro">
@@ -40,4 +41,11 @@
        deviations. -->
   <xacro:property name="lidar_noise_stddev" value="0.01"/>
+  <!-- A low-cost MEMS IMU, of which the filters use only the gyro. Its noise per sample at 100 Hz
+       comes from a rate noise density of about 0.005 deg/s/sqrt(Hz); its bias is what is left after
+       a start-up calibration, drawn anew at every start. -->
+  <xacro:property name="imu_rate" value="100"/>
+  <xacro:property name="gyro_noise_stddev" value="0.0009"/>  <!-- rad/s -->
+  <xacro:property name="gyro_bias_stddev" value="0.001"/>  <!-- rad/s -->
+  <xacro:property name="accel_noise_stddev" value="0.02"/>  <!-- m/s^2 -->
   <material name="body"><color rgba="0.15 0.35 0.6 1"/></material>
   <material name="dark"><color rgba="0.1 0.1 0.1 1"/></material>
@@ -229,4 +237,43 @@
     </sensor>
   </gazebo>
+  <!-- ===================== IMU ===================== -->
+  <joint name="imu_joint" type="fixed">
+    <parent link="base_link"/>
+    <child link="imu_link"/>
+    <origin xyz="0 0 0" rpy="0 0 0"/>
+  </joint>
+  <link name="imu_link">
+    <xacro:box_inertia mass="0.01" x="0.02" y="0.02" z="0.005"/>
+  </link>
+  <xacro:macro name="imu_noise" params="stddev bias_stddev">
+    <noise type="gaussian">
+      <mean>0</mean>
+      <stddev>${stddev}</stddev>
+      <bias_mean>0</bias_mean>
+      <bias_stddev>${bias_stddev}</bias_stddev>
+    </noise>
+  </xacro:macro>
+  <gazebo reference="imu_link">
+    <sensor name="imu" type="imu">
+      <always_on>true</always_on>
+      <update_rate>${imu_rate}</update_rate>
+      <topic>/imu</topic>
+      <gz_frame_id>imu_link</gz_frame_id>
+      <imu>
+        <!-- A real gyro gives no orientation of its own; Gazebo's would be the true one. -->
+        <enable_orientation>false</enable_orientation>
+        <angular_velocity>
+          <x><xacro:imu_noise stddev="${gyro_noise_stddev}" bias_stddev="${gyro_bias_stddev}"/></x>
+          <y><xacro:imu_noise stddev="${gyro_noise_stddev}" bias_stddev="${gyro_bias_stddev}"/></y>
+          <z><xacro:imu_noise stddev="${gyro_noise_stddev}" bias_stddev="${gyro_bias_stddev}"/></z>
+        </angular_velocity>
+        <linear_acceleration>
+          <x><xacro:imu_noise stddev="${accel_noise_stddev}" bias_stddev="0"/></x>
+          <y><xacro:imu_noise stddev="${accel_noise_stddev}" bias_stddev="0"/></y>
+          <z><xacro:imu_noise stddev="${accel_noise_stddev}" bias_stddev="0"/></z>
+        </linear_acceleration>
+      </imu>
+    </sensor>
+  </gazebo>
   <!-- ===================== Gazebo systems ===================== -->
   <gazebo>
@@ -237,6 +284,8 @@
       <wheel_radius>${wheel_radius}</wheel_radius>
       <topic>/cmd_vel</topic>
-      <odom_topic>/odom</odom_topic>
-      <tf_topic>/tf</tf_topic>
+      <!-- Gazebo's own wheel odometry is nearly exact: noisy_odometry adds the drift a real robot
+           has, and the local filter publishes odom -> base_footprint, so none of this reaches /tf. -->
+      <odom_topic>/sim/wheel_odometry</odom_topic>
+      <tf_topic>/sim/wheel_odometry/tf</tf_topic>
       <frame_id>odom</frame_id>
       <child_frame_id>base_footprint</child_frame_id>

Commit message: fix: make the simulated markers and base behave like real ones
Markers are printed on one face only and tilted wall markers sit clear of the wall. The base's speed and acceleration limits apply in both directions, and a launch argument switches the wheels' collision shape between a sphere and a cylinder.

File: aruco_world/urdf/camera_bot.urdf.xacro (robot description, xacro)
@@ -10,4 +10,7 @@
 -->
 <robot name="camera_bot" xmlns:xacro="http://www.ros.org/wiki/xacro">
+  <!-- The wheels' collision shape: "sphere" (the default, see the wheel macro) or "cylinder", the
+       shape they are drawn as, kept to compare the two. -->
+  <xacro:arg name="wheel_collision" default="sphere"/>
   <!-- Dimensions in metres, masses in kilograms -->
   <xacro:property name="body_length" value="0.36"/>
@@ -31,4 +34,9 @@
   <xacro:property name="lidar_mass" value="0.1"/>
   <xacro:property name="mast_radius" value="0.01"/>
+  <!-- What the base can do, in m/s, rad/s and their rates of change -->
+  <xacro:property name="max_speed" value="0.6"/>
+  <xacro:property name="max_turn_rate" value="1.5"/>
+  <xacro:property name="max_acceleration" value="1.0"/>
+  <xacro:property name="max_turn_acceleration" value="2.0"/>
   <!-- A low-cost 360-degree time-of-flight lidar, from the datasheets of two common ones: 5,000
        samples per second at 10 turns per second, so 500 rays 0.72 degrees apart. Where they
@@ -130,5 +138,10 @@
            touches at one point, right under the wheel's centre. -->
       <collision>
-        <geometry><sphere radius="${wheel_radius}"/></geometry>
+        <xacro:if value="${'$(arg wheel_collision)' == 'sphere'}">
+          <geometry><sphere radius="${wheel_radius}"/></geometry>
+        </xacro:if>
+        <xacro:if value="${'$(arg wheel_collision)' == 'cylinder'}">
+          <geometry><cylinder radius="${wheel_radius}" length="${wheel_width}"/></geometry>
+        </xacro:if>
       </collision>
     </link>
@@ -291,8 +304,15 @@
       <child_frame_id>base_footprint</child_frame_id>
       <odom_publish_frequency>30</odom_publish_frequency>
-      <max_linear_velocity>0.6</max_linear_velocity>
-      <max_angular_velocity>1.5</max_angular_velocity>
-      <max_linear_acceleration>1.0</max_linear_acceleration>
-      <max_angular_acceleration>2.0</max_angular_acceleration>
+      <!-- Every limit on both sides: Gazebo's speed limiter leaves a bound it is not given at
+           infinity, so with the maximums alone, braking, reversing and turning right would be
+           instantaneous and unbounded. -->
+      <max_linear_velocity>${max_speed}</max_linear_velocity>
+      <min_linear_velocity>${-max_speed}</min_linear_velocity>
+      <max_angular_velocity>${max_turn_rate}</max_angular_velocity>
+      <min_angular_velocity>${-max_turn_rate}</min_angular_velocity>
+      <max_linear_acceleration>${max_acceleration}</max_linear_acceleration>
+      <min_linear_acceleration>${-max_acceleration}</min_linear_acceleration>
+      <max_angular_acceleration>${max_turn_acceleration}</max_angular_acceleration>
+      <min_angular_acceleration>${-max_turn_acceleration}</min_angular_acceleration>
     </plugin>
     <plugin filename="gz-sim-joint-state-publisher-system"
